Commit message: nothing

File: assets/urdf/dual_robot.urdf (robot description, URDF)
Before this commit: robot dual_robot, 46 links, 45 joints
Links:
- removed link top_camera_realsense_accel_frame
- removed link top_camera_realsense_accel_optical_frame
- removed link top_camera_realsense_bottom_screw_frame
- removed link top_camera_realsense_color_frame
- removed link top_camera_realsense_color_optical_frame
- removed link top_camera_realsense_depth_frame
- removed link top_camera_realsense_depth_optical_frame
- removed link top_camera_realsense_gyro_frame
- removed link top_camera_realsense_gyro_optical_frame
- removed link top_camera_realsense_infra1_frame
- removed link top_camera_realsense_infra1_optical_frame
- removed link top_camera_realsense_infra2_frame
- removed link top_camera_realsense_infra2_optical_frame
- removed link top_camera_realsense_link
Joints:
- removed joint top_camera_realsense_accel_joint
- removed joint top_camera_realsense_accel_optical_joint
- removed joint top_camera_realsense_color_joint
- removed joint top_camera_realsense_color_optical_joint
- removed joint top_camera_realsense_depth_joint
- removed joint top_camera_realsense_depth_optical_joint
- removed joint top_camera_realsense_gyro_joint
- removed joint top_camera_realsense_gyro_optical_joint
- removed joint top_camera_realsense_infra1_joint
- removed joint top_camera_realsense_infra1_optical_joint
- removed joint top_camera_realsense_infra2_joint
- removed joint top_camera_realsense_infra2_optical_joint
- removed joint top_camera_realsense_joint
- removed joint top_camera_realsense_link_joint

Commit message: nothing

File: assets/urdf/dual_robot.urdf (robot description, URDF)
Before this commit: robot dual_robot, 32 links, 31 joints
Joints:
- joint desk_base_virtual_joint: origin xyz=0 0 0.80 rpy=0 0 0  -> xyz=0 0 0.725 rpy=0 0 0 

Commit message: nothing

File: assets/urdf/dual_robot.urdf (robot description, URDF)
Before this commit: robot dual_robot, 32 links, 31 joints
Links:
- removed link left_base
- removed link left_flange
- removed link left_tool0
- removed link right_base
- removed link right_flange
- removed link right_tool0
- added link left_arm_left_inner_finger, mass 0.0104003125914103; collision mesh filename=../dual_description/meshes/collision/robotiq/robotiq_arg2f_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 scale=0.001 0.001 0.001; visual mesh filename=../dual_description/meshes/visual/robotiq/robotiq_arg2f_85_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 scale=0.001 0.001 0.001
- added link left_arm_left_inner_finger_pad, mass 1.; collision box size=0.022 0.00635 0.0375; visual box size=0.022 0.00635 0.0375
- added link left_arm_left_inner_knuckle, mass 0.0271177346495152; collision mesh filename=../dual_description/meshes/collision/robotiq/robotiq_arg2f_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 scale=0.001 0.001 0.001; visual mesh filename=../dual_description/meshes/visual/robotiq/robotiq_arg2f_85_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 scale=0.001 0.001 0.001
- added link left_arm_left_outer_finger, mass 0.022614240507152; collision mesh filename=../dual_description/meshes/collision/robotiq/robotiq_arg2f_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 scale=0.001 0.001 0.001; visual mesh filename=../dual_description/meshes/visual/robotiq/robotiq_arg2f_85_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 scale=0.001 0.001 0.001
- added link left_arm_left_outer_knuckle, mass 0.00853198276973456; collision mesh filename=../dual_description/meshes/collision/robotiq/robotiq_arg2f_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 scale=0.001 0.001 0.001; visual mesh filename=../dual_description/meshes/visual/robotiq/robotiq_arg2f_85_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 scale=0.001 0.001 0.001
- added link left_arm_right_inner_finger, mass 0.0104003125914103; collision mesh filename=../dual_description/meshes/collision/robotiq/robotiq_arg2f_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 scale=0.001 0.001 0.001; visual mesh filename=../dual_description/meshes/visual/robotiq/robotiq_arg2f_85_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 scale=0.001 0.001 0.001
- added link left_arm_right_inner_finger_pad, mass 1; collision box size=0.022 0.00635 0.0375; visual box size=0.022 0.00635 0.0375
- added link left_arm_right_inner_knuckle, mass 0.0271177346495152; collision mesh filename=../dual_description/meshes/collision/robotiq/robotiq_arg2f_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 scale=0.001 0.001 0.001; visual mesh filename=../dual_description/meshes/visual/robotiq/robotiq_arg2f_85_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 scale=0.001 0.001 0.001
- added link left_arm_right_outer_finger, mass 0.022614240507152; collision mesh filename=../dual_description/meshes/collision/robotiq/robotiq_arg2f_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 scale=0.001 0.001 0.001; visual mesh filename=../dual_description/meshes/visual/robotiq/robotiq_arg2f_85_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 scale=0.001 0.001 0.001
- added link left_arm_right_outer_knuckle, mass 0.00853198276973456; collision mesh filename=../dual_description/meshes/collision/robotiq/robotiq_arg2f_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 scale=0.001 0.001 0.001; visual mesh filename=../dual_description/meshes/visual/robotiq/robotiq_arg2f_85_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 scale=0.001 0.001 0.001
- added link left_robotiq_arg2f_base_link, mass 0.22652; collision mesh filename=../dual_description/meshes/collision/robotiq/robotiq_arg2f_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; visual mesh filename=../dual_description/meshes/visual/robotiq/robotiq_arg2f_85_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 scale=0.001 0.001 0.001
- added link right_arm_left_inner_finger, mass 0.0104003125914103; collision mesh filename=../dual_description/meshes/collision/robotiq/robotiq_arg2f_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 scale=0.001 0.001 0.001; visual mesh filename=../dual_description/meshes/visual/robotiq/robotiq_arg2f_85_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 scale=0.001 0.001 0.001
- added link right_arm_left_inner_finger_pad, mass 1.; collision box size=0.022 0.00635 0.0375; visual box size=0.022 0.00635 0.0375
- added link right_arm_left_inner_knuckle, mass 0.0271177346495152; collision mesh filename=../dual_description/meshes/collision/robotiq/robotiq_arg2f_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 scale=0.001 0.001 0.001; visual mesh filename=../dual_description/meshes/visual/robotiq/robotiq_arg2f_85_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 scale=0.001 0.001 0.001
- added link right_arm_left_outer_finger, mass 0.022614240507152; collision mesh filename=../dual_description/meshes/collision/robotiq/robotiq_arg2f_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 scale=0.001 0.001 0.001; visual mesh filename=../dual_description/meshes/visual/robotiq/robotiq_arg2f_85_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 scale=0.001 0.001 0.001
- added link right_arm_left_outer_knuckle, mass 0.00853198276973456; collision mesh filename=../dual_description/meshes/collision/robotiq/robotiq_arg2f_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 scale=0.001 0.001 0.001; visual mesh filename=../dual_description/meshes/visual/robotiq/robotiq_arg2f_85_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 scale=0.001 0.001 0.001
- added link right_arm_right_inner_finger, mass 0.0104003125914103; collision mesh filename=../dual_description/meshes/collision/robotiq/robotiq_arg2f_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 scale=0.001 0.001 0.001; visual mesh filename=../dual_description/meshes/visual/robotiq/robotiq_arg2f_85_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 scale=0.001 0.001 0.001
- added link right_arm_right_inner_finger_pad, mass 1; collision box size=0.022 0.00635 0.0375; visual box size=0.022 0.00635 0.0375
- added link right_arm_right_inner_knuckle, mass 0.0271177346495152; collision mesh filename=../dual_description/meshes/collision/robotiq/robotiq_arg2f_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 scale=0.001 0.001 0.001; visual mesh filename=../dual_description/meshes/visual/robotiq/robotiq_arg2f_85_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 scale=0.001 0.001 0.001
- added link right_arm_right_outer_finger, mass 0.022614240507152; collision mesh filename=../dual_description/meshes/collision/robotiq/robotiq_arg2f_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 scale=0.001 0.001 0.001; visual mesh filename=../dual_description/meshes/visual/robotiq/robotiq_arg2f_85_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 scale=0.001 0.001 0.001
- added link right_arm_right_outer_knuckle, mass 0.00853198276973456; collision mesh filename=../dual_description/meshes/collision/robotiq/robotiq_arg2f_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 scale=0.001 0.001 0.001; visual mesh filename=../dual_description/meshes/visual/robotiq/robotiq_arg2f_85_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 scale=0.001 0.001 0.001
- added link right_robotiq_arg2f_base_link, mass 0.22652; collision mesh filename=../dual_description/meshes/collision/robotiq/robotiq_arg2f_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; visual mesh filename=../dual_description/meshes/visual/robotiq/robotiq_arg2f_85_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 scale=0.001 0.001 0.001
Joints:
- removed joint left_base_link-base_fixed_joint
- removed joint left_flange-tool0
- removed joint left_wrist_3-flange
- removed joint right_base_link-base_fixed_joint
- removed joint right_flange-tool0
- removed joint right_wrist_3-flange
- added joint left_arm_left_inner_finger_joint: type revolute, parent left_arm_left_outer_finger, child left_arm_left_inner_finger, origin xyz=0 0.0061 0.0471 rpy=0 0 0, axis 1 0 0, limit lower=-0.8757 upper=0 effort=1000 velocity=2.0, mimic joint=finger_joint multiplier=-1 offset=0
- added joint left_arm_left_inner_finger_pad_joint: type fixed, parent left_arm_left_inner_finger, child left_arm_left_inner_finger_pad, origin xyz=0 -0.0220203446692936 0.03242 rpy=0 0 0, axis 0 0 1
- added joint left_arm_left_inner_knuckle_joint: type revolute, parent left_robotiq_arg2f_base_link, child left_arm_left_inner_knuckle, origin xyz=0 -0.0127 0.06142 rpy=0 0 3.14159265359, axis 1 0 0, limit lower=0 upper=0.8757 effort=1000 velocity=2.0, mimic joint=finger_joint multiplier=1 offset=0
- added joint left_arm_left_outer_finger_joint: type fixed, parent left_arm_left_outer_knuckle, child left_arm_left_outer_finger, origin xyz=0 0.0315 -0.0041 rpy=0 0 0, axis 1 0 0
- added joint left_arm_right_inner_finger_joint: type revolute, parent left_arm_right_outer_finger, child left_arm_right_inner_finger, origin xyz=0 0.0061 0.0471 rpy=0 0 0, axis 1 0 0, limit lower=-0.8757 upper=0 effort=1000 velocity=2.0, mimic joint=finger_joint multiplier=-1 offset=0
- added joint left_arm_right_inner_finger_pad_joint: type fixed, parent left_arm_right_inner_finger, child left_arm_right_inner_finger_pad, origin xyz=0 -0.0220203446692936 0.03242 rpy=0 0 0, axis 0 0 1
- added joint left_arm_right_inner_knuckle_joint: type revolute, parent left_robotiq_arg2f_base_link, child left_arm_right_inner_knuckle, origin xyz=0 0.0127 0.06142 rpy=0 0 0.0, axis 1 0 0, limit lower=0 upper=0.8757 effort=1000 velocity=2.0, mimic joint=finger_joint multiplier=1 offset=0
- added joint left_arm_right_outer_finger_joint: type fixed, parent left_arm_right_outer_knuckle, child left_arm_right_outer_finger, origin xyz=0 0.0315 -0.0041 rpy=0 0 0, axis 1 0 0
- added joint left_arm_right_outer_knuckle_joint: type revolute, parent left_robotiq_arg2f_base_link, child left_arm_right_outer_knuckle, origin xyz=0 0.0306011 0.054904 rpy=0 0 0, axis 1 0 0, limit lower=0 upper=0.81 effort=1000 velocity=2.0, mimic joint=finger_joint multiplier=1 offset=0
- added joint left_ee_joint: type fixed, parent left_wrist_3_link, child left_robotiq_arg2f_base_link, origin xyz=0 0 0 rpy=0 0 -1.5707963267948966
- added joint left_finger_joint: type revolute, parent left_robotiq_arg2f_base_link, child left_arm_left_outer_knuckle, origin xyz=0 -0.0306011 0.054904 rpy=0 0 3.14159265359, axis 1 0 0, limit lower=0 upper=0.8 effort=1000 velocity=2.0
- added joint right_arm_left_inner_finger_joint: type revolute, parent right_arm_left_outer_finger, child right_arm_left_inner_finger, origin xyz=0 0.0061 0.0471 rpy=0 0 0, axis 1 0 0, limit lower=-0.8757 upper=0 effort=1000 velocity=2.0, mimic joint=finger_joint multiplier=-1 offset=0
- added joint right_arm_left_inner_finger_pad_joint: type fixed, parent right_arm_left_inner_finger, child right_arm_left_inner_finger_pad, origin xyz=0 -0.0220203446692936 0.03242 rpy=0 0 0, axis 0 0 1
- added joint right_arm_left_inner_knuckle_joint: type revolute, parent right_robotiq_arg2f_base_link, child right_arm_left_inner_knuckle, origin xyz=0 -0.0127 0.06142 rpy=0 0 3.14159265359, axis 1 0 0, limit lower=0 upper=0.8757 effort=1000 velocity=2.0, mimic joint=finger_joint multiplier=1 offset=0
- added joint right_arm_left_outer_finger_joint: type fixed, parent right_arm_left_outer_knuckle, child right_arm_left_outer_finger, origin xyz=0 0.0315 -0.0041 rpy=0 0 0, axis 1 0 0
- added joint right_arm_right_inner_finger_joint: type revolute, parent right_arm_right_outer_finger, child right_arm_right_inner_finger, origin xyz=0 0.0061 0.0471 rpy=0 0 0, axis 1 0 0, limit lower=-0.8757 upper=0 effort=1000 velocity=2.0, mimic joint=finger_joint multiplier=-1 offset=0
- added joint right_arm_right_inner_finger_pad_joint: type fixed, parent right_arm_right_inner_finger, child right_arm_right_inner_finger_pad, origin xyz=0 -0.0220203446692936 0.03242 rpy=0 0 0, axis 0 0 1
- added joint right_arm_right_inner_knuckle_joint: type revolute, parent right_robotiq_arg2f_base_link, child right_arm_right_inner_knuckle, origin xyz=0 0.0127 0.06142 rpy=0 0 0.0, axis 1 0 0, limit lower=0 upper=0.8757 effort=1000 velocity=2.0, mimic joint=finger_joint multiplier=1 offset=0
- added joint right_arm_right_outer_finger_joint: type fixed, parent right_arm_right_outer_knuckle, child right_arm_right_outer_finger, origin xyz=0 0.0315 -0.0041 rpy=0 0 0, axis 1 0 0
- added joint right_arm_right_outer_knuckle_joint: type revolute, parent right_robotiq_arg2f_base_link, child right_arm_right_outer_knuckle, origin xyz=0 0.0306011 0.054904 rpy=0 0 0, axis 1 0 0, limit lower=0 upper=0.81 effort=1000 velocity=2.0, mimic joint=finger_joint multiplier=1 offset=0
- added joint right_ee_joint: type fixed, parent right_wrist_3_link, child right_robotiq_arg2f_base_link, origin xyz=0 0 0 rpy=0 0 -1.5707963267948966
- added joint right_finger_joint: type revolute, parent right_robotiq_arg2f_base_link, child right_arm_left_outer_knuckle, origin xyz=0 -0.0306011 0.054904 rpy=0 0 3.14159265359, axis 1 0 0, limit lower=0 upper=0.8 effort=1000 velocity=2.0

Commit message: nothing

File: assets/urdf/dual_robot.urdf (robot description, URDF)
Before this commit: robot dual_robot, 48 links, 47 joints
Links:
- removed link base_left_virtual_link
- removed link base_right_virtual_link
- removed link left_base_link
- removed link right_base_link
- removed link top_camera_virtual_link
- removed link top_mid_virtual_link
Joints:
- removed joint base_left_virtual_joint
- removed joint base_right_virtual_joint
- removed joint left_base_link-base_link_inertia
- removed joint right_base_link-base_link_inertia
- removed joint top_camera_virtual_joint
- removed joint top_mid_virtual_joint
- joint left_fixed: child left_base_link -> left_base_link_inertia; origin xyz=0 0 0 rpy=0 0 3.141592653 -> xyz=0 0.1747487373415 0.6411091270347 rpy=-2.35619449019234 0 0; parent base_left_virtual_link -> body_base_link
- joint right_fixed: child right_base_link -> right_base_link_inertia; origin xyz=0 0 0 rpy=0 0 1.57  -> xyz=0 -0.174748737341515 0.641109127034685 rpy=3.14159265358979 0.785398163397448 1.57 ; parent base_right_virtual_link -> body_base_link

Commit message: nothing

File: assets/urdf/dual_robot.urdf (robot description, URDF)
Before this commit: robot dual_robot, 42 links, 41 joints
Joints:
- joint right_fixed: origin xyz=0 -0.174748737341515 0.641109127034685 rpy=3.14159265358979 0.785398163397448 1.57  -> xyz=0 -0.174748737341515 0.641109127034685 rpy=2.35619449019234 0 0 

Commit message: big change

File: assets/urdf/dual_robot.urdf (robot description, URDF)
Before this commit: robot dual_robot, 42 links, 41 joints
Joints:
- joint left_arm_left_inner_finger_joint: mimic joint=finger_joint multiplier=-1 offset=0 -> joint=left_finger_joint multiplier=-1 offset=0
- joint left_arm_left_inner_knuckle_joint: mimic joint=finger_joint multiplier=1 offset=0 -> joint=left_finger_joint multiplier=1 offset=0
- joint left_arm_right_inner_finger_joint: mimic joint=finger_joint multiplier=-1 offset=0 -> joint=left_finger_joint multiplier=-1 offset=0
- joint left_arm_right_inner_knuckle_joint: mimic joint=finger_joint multiplier=1 offset=0 -> joint=left_finger_joint multiplier=1 offset=0
- joint left_arm_right_outer_knuckle_joint: mimic joint=finger_joint multiplier=1 offset=0 -> joint=left_finger_joint multiplier=1 offset=0
- joint left_wrist_1_joint: origin xyz=-0.3922 0 0.1333 rpy=0 0 0 -> xyz=-0.3922 0 0.1333 rpy=0 0 -1.5707963267948966
- joint right_arm_left_inner_finger_joint: mimic joint=finger_joint multiplier=-1 offset=0 -> joint=right_finger_joint multiplier=-1 offset=0
- joint right_arm_left_inner_knuckle_joint: mimic joint=finger_joint multiplier=1 offset=0 -> joint=right_finger_joint multiplier=1 offset=0
- joint right_arm_right_inner_finger_joint: mimic joint=finger_joint multiplier=-1 offset=0 -> joint=right_finger_joint multiplier=-1 offset=0
- joint right_arm_right_inner_knuckle_joint: mimic joint=finger_joint multiplier=1 offset=0 -> joint=right_finger_joint multiplier=1 offset=0
- joint right_arm_right_outer_knuckle_joint: mimic joint=finger_joint multiplier=1 offset=0 -> joint=right_finger_joint multiplier=1 offset=0
- joint right_ee_joint: origin xyz=0 0 0 rpy=0 0 -1.5707963267948966 -> xyz=0 0 0 rpy=0 0 1.5707963267948966
- joint right_shoulder_lift_joint: origin xyz=0 0 0 rpy=1.570796327 0 0 -> xyz=0 0 0 rpy=1.570796327 3.141592653589793 0
- joint right_shoulder_pan_joint: origin xyz=0 0 0.1625 rpy=0 0 0 -> xyz=0 0 0.1625 rpy=0 0 3.141592653589793
- joint right_wrist_1_joint: origin xyz=-0.3922 0 0.1333 rpy=0 0 0 -> xyz=-0.3922 0 0.1333 rpy=0 0 -1.5707963267948966
